File: 2021本ロボメインシールド.kicad_pcb (KiCad board)
At the start: 2 copper layers, 165.1 x 92.7 mm, 53 parts, among them P1 Digital, P2 Power, P3 Analog, P4 Analog, P5 PWM, P6 PWM, P7 Communication, SW1 SW_Push

Commit message: ver1.2
Routing:
- net SS7: track 212.4 -> 222.7 mm
- net RX1: track 48.5 -> 56.6 mm
- net TX1: track 45.1 -> 51.7 mm
- net SS10: track 298.5 -> 304.2 mm
- net SS6: track 180.1 -> 183.7 mm
- net SS5: track 154.4 -> 157.6 mm
- net SS9: track 273.4 -> 275.7 mm
- net GND: track 11.1 -> 8.89 mm, vias 1 -> 0
- net SS4: track 127.9 -> 129.6 mm
- net SS8: track 247.7 -> 248.9 mm
- net MOSI: track 273.9 -> 272.9 mm
- net MISO: track 261.3 -> 262.0 mm
- net +3V3: track 135.6 -> 136.2 mm, vias 0 -> 2
Other:
- board text added: "NIT Toyota College ROBOCON A team Main shield for Arduino Mega ver1.2 Designed by Taichi Kondo 2021/05/29"
- board text removed: "Main shield for Arduino Mega ver1.0 2021/06/27 Designed by Taichi Kondo"

Commit message: ver1.3 stepping10->9
Parts:
- removed STEP_SPI10: Conn_02x05_Odd_Even, Connector_IDC:IDC-Header_2x05_P2.54mm_Vertical
Connections:
- P1 pad 7: /48 -> BUSY8
- P1 pad 9: /46 -> BUSY9
- P3 pad 1: SS10 -> SS9
- P3 pad 2: SS9 -> SS8
- P3 pad 3: SS8 -> SS7
- P3 pad 4: SS7 -> SS6
- P3 pad 5: SS6 -> SS5
- P3 pad 6: SS5 -> SS4
- P3 pad 7: SS4 -> SS3
- P3 pad 8: SS3 -> SS2
- P4 pad 1: SS2 -> SS1
- P4 pad 2: SS1 -> BUSY1
- P4 pad 3: /A10 -> BUSY2
- P4 pad 4: /A11 -> BUSY3
- P4 pad 5: /A12 -> BUSY4
- P4 pad 6: /A13 -> BUSY5
- P4 pad 7: /A14 -> BUSY6
- P4 pad 8: /A15 -> BUSY7
- STEP_SPI1 pad 1: Net-(STEP_SPI1-Pad1) -> BUSY1
- STEP_SPI2 pad 1: Net-(STEP_SPI2-Pad1) -> BUSY2
- STEP_SPI3 pad 1: Net-(STEP_SPI3-Pad1) -> BUSY3
- STEP_SPI4 pad 1: Net-(STEP_SPI4-Pad1) -> BUSY4
- STEP_SPI5 pad 1: Net-(STEP_SPI5-Pad1) -> BUSY5
- STEP_SPI6 pad 1: Net-(STEP_SPI6-Pad1) -> BUSY6
- STEP_SPI7 pad 1: Net-(STEP_SPI7-Pad1) -> BUSY7
- STEP_SPI8 pad 1: Net-(STEP_SPI8-Pad1) -> BUSY8
- STEP_SPI9 pad 1: Net-(STEP_SPI9-Pad1) -> BUSY9
Routing:
- net SS10: track 304.2 -> 0.00 mm, vias 1 -> 0
- net BUSY7: track 0.00 -> 167.5 mm
- net BUSY6: track 0.00 -> 147.6 mm
- net BUSY5: track 0.00 -> 128.7 mm
- net BUSY4: track 0.00 -> 109.9 mm
- net SS8: track 248.9 -> 339.5 mm
- net BUSY3: track 0.00 -> 88.1 mm
- net BUSY8: track 0.00 -> 85.4 mm, vias 0 -> 1
- net BUSY9: track 0.00 -> 82.7 mm, vias 0 -> 2
- net BUSY2: track 0.00 -> 66.8 mm
- net GND: track 8.89 -> 55.9 mm, vias 0 -> 7
- net BUSY1: track 0.00 -> 46.6 mm
- net MOSI: track 272.9 -> 237.0 mm, vias 0 -> 9
- net MISO: track 262.0 -> 239.2 mm
- net SCK: track 278.1 -> 255.8 mm
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